Commit message: new urdf from xacro

File: awtube31814v2/xacro/awtube31814v2.urdf (robot description, URDF)
Before this commit: robot awtube31814v2, 7 links, 6 joints
Joints:
- joint awtube_joint3: axis 0 0 -1 -> 0 0 1; limit lower=-4.71 upper=1.57 effort=350 velocity=1.24 -> lower=-4.71 upper=4.71 effort=350 velocity=1.24
- joint awtube_joint5: limit lower=-1.6 upper=4.71 effort=145 velocity=2.71 -> lower=-4.71 upper=4.71 effort=145 velocity=2.71
