Commit message: joint limits from yaml

File: xacro/robofox.urdf.xacro (robot description, xacro)
@@ -5,8 +5,11 @@
     <xacro:arg name="physical_params_file"
         default="$(find ibt_ros2_description)/config/$(arg robofox_type)/physical_parameters.yaml" />
+    <xacro:arg name="joint_limits_file"
+        default="$(find ibt_ros2_description)/config/$(arg robofox_type)/joint_limits.yaml" />
     <xacro:include filename="$(find ibt_ros2_description)/xacro/robofox.xacro" />
     <xacro:robofox
         prefix="$(arg prefix)"
         physical_params_file="$(arg physical_params_file)"
+        joint_limits_file="$(arg joint_limits_file)"
         robofox_type="$(arg robofox_type)"
     >

File: xacro/robofox.xacro (robot description, xacro)
@@ -8,5 +8,6 @@
     connected_to:=''
     *origin
-    physical_params_file"
+    physical_params_file
+    joint_limits_file"
   >
     <xacro:property name="physical_params"
@@ -16,4 +17,10 @@
     <xacro:property name="sec_inertia_parameters"
       value="${config_physical_parameters['inertial_parameters']}" />
+    <xacro:property name="joint_limits"
+      value="${joint_limits_file}"/>
+    <xacro:property name="config_joint_limits"
+      value="${xacro.load_yaml(joint_limits)}" />
+    <xacro:property name="sec_limits"
+      value="${config_joint_limits['joint_limits']}"/>
     <!-- INERTIA PARAMETERS -->
     <!-- mass -->
@@ -191,8 +198,8 @@
         xyz="0 0 -1" />
       <limit
-        lower="-${pi}"
-        upper="${pi}"
-        effort="600"
-        velocity="1.2436" />
+        lower="${sec_limits['joint1']['min_position']}"
+        upper="${sec_limits['joint1']['max_position']}"
+        effort="${sec_limits['joint1']['max_effort']}"
+        velocity="${sec_limits['joint1']['max_velocity']}" />
       <dynamics
         damping="1"
@@ -251,8 +258,8 @@
         xyz="0 0 -1" />
       <limit
-        lower="-${pi}"
-        upper="${pi}"
-        effort="690"
-        velocity="0.86" />
+        lower="${sec_limits['joint2']['min_position']}"
+        upper="${sec_limits['joint2']['max_position']}"
+        effort="${sec_limits['joint2']['max_effort']}"
+        velocity="${sec_limits['joint2']['max_velocity']}" />
       <dynamics
         damping="1"
@@ -311,8 +318,8 @@
         xyz="0 0 -1" />
       <limit
-        lower="-4.71"
-        upper="4.71"
-        effort="350"
-        velocity="1.24" />
+        lower="${sec_limits['joint3']['min_position']}"
+        upper="${sec_limits['joint3']['max_position']}"
+        effort="${sec_limits['joint3']['max_effort']}"
+        velocity="${sec_limits['joint3']['max_velocity']}" />
       <dynamics
         damping="1"
@@ -371,8 +378,8 @@
         xyz="0 0 -1" />
       <limit
-        lower="-8.0"
-        upper="8.0"
-        effort="145"
-        velocity="2.71" />
+        lower="${sec_limits['joint4']['min_position']}"
+        upper="${sec_limits['joint4']['max_position']}"
+        effort="${sec_limits['joint4']['max_effort']}"
+        velocity="${sec_limits['joint4']['max_velocity']}" />
       <dynamics
         damping="1"
@@ -431,8 +438,8 @@
         xyz="0 0 -1" />
       <limit
-        lower="-4.71"
-        upper="4.71"
-        effort="145"
-        velocity="2.71" />
+        lower="${sec_limits['joint5']['min_position']}"
+        upper="${sec_limits['joint5']['max_position']}"
+        effort="${sec_limits['joint5']['max_effort']}"
+        velocity="${sec_limits['joint5']['max_velocity']}" />
       <dynamics
         damping="1"
@@ -491,8 +498,8 @@
         xyz="0 0 -1" />
       <limit
-        lower="-8.0"
-        upper="8.0"
-        effort="85"
-        velocity="3.61" />
+        lower="${sec_limits['joint6']['min_position']}"
+        upper="${sec_limits['joint6']['max_position']}"
+        effort="${sec_limits['joint6']['max_effort']}"
+        velocity="${sec_limits['joint6']['max_velocity']}" />
       <dynamics
         damping="1"
