Commit message: fixed joint_limits

File: xacro/robofox.xacro (robot description, xacro)
@@ -127,6 +127,6 @@
           rpy="0 0 0" />
         <geometry>
-          <mesh
-            filename="package://ibt_ros2_description/meshes/${robofox_type}/visual/baselink.STL" />
+          <!-- <mesh
+            filename="package://ibt_ros2_description/meshes/${robofox_type}/visual/baselink.STL" /> -->
         </geometry>
         <material
@@ -166,6 +166,6 @@
           rpy="0 0 0" />
         <geometry>
-          <mesh
-            filename="package://ibt_ros2_description/meshes/${robofox_type}/visual/link1.STL" />
+          <!-- <mesh
+            filename="package://ibt_ros2_description/meshes/${robofox_type}/visual/link1.STL" /> -->
         </geometry>
         <material

Commit message: mesh completed

File: xacro/robofox.xacro (robot description, xacro)
@@ -127,20 +127,20 @@
           rpy="0 0 0" />
         <geometry>
-          <!-- <mesh
-            filename="package://ibt_ros2_description/meshes/${robofox_type}/visual/baselink.STL" /> -->
-        </geometry>
-        <material
-          name="">
-          <color
-            rgba="0.79216 0.81961 0.93333 1" />
-        </material>
-      </visual>
-      <collision>
-        <origin
-          xyz="0 0 0"
-          rpy="0 0 0" />
-        <geometry>
-          <!-- <mesh
-            filename="package://ibt_ros2_description/meshes/${robofox_type}/collision/baselink.STL" /> -->
+          <mesh
+            filename="package://ibt_ros2_description/meshes/${robofox_type}/visual/base_link.STL" />
+        </geometry>
+        <material
+          name="">
+          <color
+            rgba="0.30 0.30 0.30 1" />
+        </material>
+      </visual>
+      <collision>
+        <origin
+          xyz="0 0 0"
+          rpy="0 0 0" />
+        <geometry>
+          <mesh
+            filename="package://ibt_ros2_description/meshes/${robofox_type}/visual/base_link.STL" />
         </geometry>
       </collision>
@@ -163,23 +163,23 @@
       <visual>
         <origin
-          xyz="0 0 -0.09"
-          rpy="0 0 0" />
-        <geometry>
-          <!-- <mesh
-            filename="package://ibt_ros2_description/meshes/${robofox_type}/visual/link1.STL" /> -->
-        </geometry>
-        <material
-          name="">
-          <color
-            rgba="0.79216 0.81961 0.93333 1" />
-        </material>
-      </visual>
-      <collision>
-        <origin
-          xyz="0 0 0"
-          rpy="0 0 0" />
-        <geometry>
-          <!-- <mesh
-            filename="package://ibt_ros2_description/meshes/${robofox_type}/collision/link1.STL" /> -->
+          xyz="0 0 0"
+          rpy="0 0 0" />
+        <geometry>
+          <mesh
+            filename="package://ibt_ros2_description/meshes/${robofox_type}/visual/link1.STL" />
+        </geometry>
+        <material
+          name="">
+          <color
+            rgba="0.30 0.30 0.30 1" />
+        </material>
+      </visual>
+      <collision>
+        <origin
+          xyz="0 0 0"
+          rpy="0 0 0" />
+        <geometry>
+          <mesh
+            filename="package://ibt_ros2_description/meshes/${robofox_type}/visual/link1.STL" />
         </geometry>
       </collision>
@@ -224,22 +224,22 @@
         <origin
           xyz="0 0 0"
-          rpy="0 -${pi/2} 0" />
-        <geometry>
-          <!-- <mesh
-            filename="package://ibt_ros2_description/meshes/${robofox_type}/visual/link2.STL" /> -->
-        </geometry>
-        <material
-          name="">
-          <color
-            rgba="0.79216 0.81961 0.93333 1" />
-        </material>
-      </visual>
-      <collision>
-        <origin
-          xyz="0 0 0"
-          rpy="-${pi/2.0} -${pi/2.0} 0" />
-        <geometry>
-          <!-- <mesh
-            filename="package://ibt_ros2_description/meshes/${robofox_type}/collision/link2.STL" /> -->
+          rpy="0 0 0" />
+        <geometry>
+          <mesh
+            filename="package://ibt_ros2_description/meshes/${robofox_type}/visual/link2.STL" />
+        </geometry>
+        <material
+          name="">
+          <color
+            rgba="0.30 0.30 0.30 1" />
+        </material>
+      </visual>
+      <collision>
+        <origin
+          xyz="0 0 0"
+          rpy="0 0 0" />
+        <geometry>
+          <mesh
+            filename="package://ibt_ros2_description/meshes/${robofox_type}/visual/link2.STL" />
         </geometry>
       </collision>
@@ -283,23 +283,23 @@
       <visual>
         <origin
-          xyz="0.725 0 0"
-          rpy="0 0 ${pi}" />
-        <geometry>
-          <!-- <mesh
-            filename="package://ibt_ros2_description/meshes/${robofox_type}/visual/link3.STL" /> -->
-        </geometry>
-        <material
-          name="">
-          <color
-            rgba="0.79216 0.81961 0.93333 1" />
-        </material>
-      </visual>
-      <collision>
-        <origin
-          xyz="0.725 0 0"
-          rpy="0 0 ${pi}" />
-        <geometry>
-          <!-- <mesh
-            filename="package://ibt_ros2_description/meshes/${robofox_type}/collision/link3.STL" /> -->
+          xyz="0 0 0"
+          rpy="0 0 0" />
+        <geometry>
+          <mesh
+            filename="package://ibt_ros2_description/meshes/${robofox_type}/visual/link3.STL" />
+        </geometry>
+        <material
+          name="">
+          <color
+            rgba="0.30 0.30 0.30 1" />
+        </material>
+      </visual>
+      <collision>
+        <origin
+          xyz="0 0 0"
+          rpy="0 0 0" />
+        <geometry>
+          <mesh
+            filename="package://ibt_ros2_description/meshes/${robofox_type}/visual/link3.STL" />
         </geometry>
       </collision>
@@ -344,22 +344,22 @@
         <origin
           xyz="0 0 0"
-          rpy="${pi/2.0} 0 0" />
-        <geometry>
-          <!-- <mesh
-            filename="package://ibt_ros2_description/meshes/${robofox_type}/visual/link4.STL" /> -->
-        </geometry>
-        <material
-          name="">
-          <color
-            rgba="0.79216 0.81961 0.93333 1" />
-        </material>
-      </visual>
-      <collision>
-        <origin
-          xyz="0 0 0"
-          rpy="${pi/2.0} 0 0" />
-        <geometry>
-          <!-- <mesh
-            filename="package://ibt_ros2_description/meshes/${robofox_type}/collision/link4.STL" /> -->
+          rpy="0 0 0" />
+        <geometry>
+          <mesh
+            filename="package://ibt_ros2_description/meshes/${robofox_type}/visual/link4.STL" />
+        </geometry>
+        <material
+          name="">
+          <color
+            rgba="0.30 0.30 0.30 1" />
+        </material>
+      </visual>
+      <collision>
+        <origin
+          xyz="0 0 0"
+          rpy="0 0 0" />
+        <geometry>
+          <mesh
+            filename="package://ibt_ros2_description/meshes/${robofox_type}/visual/link4.STL" />
         </geometry>
       </collision>
@@ -403,23 +403,23 @@
       <visual>
         <origin
-          xyz="0 0 0.6751"
-          rpy="-${pi/2.0} ${pi/2.0} 0" />
-        <geometry>
-          <!-- <mesh
-            filename="package://ibt_ros2_description/meshes/${robofox_type}/visual/link5.STL" /> -->
-        </geometry>
-        <material
-          name="">
-          <color
-            rgba="0.69804 0.69804 0.69804 1" />
-        </material>
-      </visual>
-      <collision>
-        <origin
-          xyz="0 0 0.6751"
-          rpy="-${pi/2.0} ${pi/2.0} 0" />
-        <geometry>
-          <!-- <mesh
-            filename="package://ibt_ros2_description/meshes/${robofox_type}/collision/link5.STL" /> -->
+          xyz="0 0 0"
+          rpy="0 0 0" />
+        <geometry>
+          <mesh
+            filename="package://ibt_ros2_description/meshes/${robofox_type}/visual/link5.STL" />
+        </geometry>
+        <material
+          name="">
+          <color
+            rgba="0.30 0.30 0.30 1" />
+        </material>
+      </visual>
+      <collision>
+        <origin
+          xyz="0 0 0"
+          rpy="0 0 0" />
+        <geometry>
+          <mesh
+            filename="package://ibt_ros2_description/meshes/${robofox_type}/visual/link5.STL" />
         </geometry>
       </collision>
@@ -463,23 +463,23 @@
       <visual>
         <origin
-          xyz="0 -0.36 0"
-          rpy="${pi/2.0} ${pi} 0" />
-        <geometry>
-          <!-- <mesh
-            filename="package://ibt_ros2_description/meshes/${robofox_type}/visual/link6.STL" /> -->
-        </geometry>
-        <material
-          name="">
-          <color
-            rgba="0.8902 0.8902 0.91373 1" />
-        </material>
-      </visual>
-      <collision>
-        <origin
-          xyz="0 -0.36 0"
-          rpy="${pi/2.0} ${pi} 0" />
-        <geometry>
-          <!-- <mesh
-            filename="package://ibt_ros2_description/meshes/${robofox_type}/collision/link6.STL" /> -->
+          xyz="0 0 0"
+          rpy="0 0 0" />
+        <geometry>
+          <mesh
+            filename="package://ibt_ros2_description/meshes/${robofox_type}/visual/link6.STL" />
+        </geometry>
+        <material
+          name="">
+          <color
+            rgba="0.30 0.30 0.30 1" />
+        </material>
+      </visual>
+      <collision>
+        <origin
+          xyz="0 0 0"
+          rpy="0 0 0" />
+        <geometry>
+          <mesh
+            filename="package://ibt_ros2_description/meshes/${robofox_type}/visual/link6.STL" />
         </geometry>
       </collision>
