Commit message: mesh parametrized

File: xacro/robofox.urdf (robot description, URDF)
Before this commit: robot robofox, 7 links, 6 joints
Links:
- link robofox_base_link: geometry collision mesh filename=package://ibt_ros2_description/meshes/robofox_type/collisio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; visual mesh filename=package://ibt_ros2_description/meshes/robofox_type/visual/b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
- link robofox_link1: geometry collision mesh filename=package://ibt_ros2_description/meshes/robofox_type/collisio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; visual mesh filename=package://ibt_ros2_description/meshes/robofox_type/visual/l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
- link robofox_link2: geometry collision mesh filename=package://ibt_ros2_description/meshes/robofox_type/collisio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; visual mesh filename=package://ibt_ros2_description/meshes/robofox_type/visual/l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
- link robofox_link3: geometry collision mesh filename=package://ibt_ros2_description/meshes/robofox_type/collisio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; visual mesh filename=package://ibt_ros2_description/meshes/robofox_type/visual/l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
- link robofox_link4: geometry collision mesh filename=package://ibt_ros2_description/meshes/robofox_type/collisio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; visual mesh filename=package://ibt_ros2_description/meshes/robofox_type/visual/l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
- link robofox_link5: geometry collision mesh filename=package://ibt_ros2_description/meshes/robofox_type/collisio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; visual mesh filename=package://ibt_ros2_description/meshes/robofox_type/visual/l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
- link robofox_link6: geometry collision mesh filename=package://ibt_ros2_description/meshes/robofox_type/collisio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; visual mesh filename=package://ibt_ros2_description/meshes/robofox_type/visual/l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

File: xacro/robofox.urdf.xacro (robot description, xacro)
@@ -1,9 +1,11 @@
 <?xml version="1.0"?>
 <robot xmlns:xacro="http://wiki.ros.org/xacro" name="robofox">
+    <xacro:arg name="prefix" default="robofox" />
     <xacro:arg name="robofox_type" default="61814v3" />
     <xacro:arg name="physical_params_file"
-        default="$(find robofox)/config/$(arg robofox_type)/physical_parameters.yaml" />
-    <xacro:include filename="$(find robofox)/xacro/robofox.xacro" />
+        default="$(find ibt_ros2_description)/config/$(arg robofox_type)/physical_parameters.yaml" />
+    <xacro:include filename="$(find ibt_ros2_description)/xacro/robofox.xacro" />
     <xacro:robofox
+        prefix="$(arg prefix)"
         physical_params_file="$(arg physical_params_file)"
     >

File: xacro/robofox.xacro (robot description, xacro)
@@ -5,4 +5,5 @@
     params="
     prefix:='robofox'
+    robofox_type:='61814v3'
     connected_to:=''
     *origin
@@ -120,5 +121,5 @@
         <geometry>
           <mesh
-            filename="package://robofox/meshes/awtube3_baselink.STL" />
+            filename="package://ibt_ros2_description/meshes/${robofox_type}/visual/baselink.STL" />
         </geometry>
         <material
@@ -134,5 +135,5 @@
         <geometry>
           <mesh
-            filename="package://robofox/meshes/controllo/awtube3_baselink.STL" />
+            filename="package://ibt_ros2_description/meshes/${robofox_type}/collision/baselink.STL" />
         </geometry>
       </collision>
@@ -159,5 +160,5 @@
         <geometry>
           <mesh
-            filename="package://robofox/meshes/awtube3_link1.STL" />
+            filename="package://ibt_ros2_description/meshes/${robofox_type}/visual/link1.STL" />
         </geometry>
         <material
@@ -173,5 +174,5 @@
         <geometry>
           <mesh
-            filename="package://robofox/meshes/controllo/awtube3_link1.STL" />
+            filename="package://ibt_ros2_description/meshes/${robofox_type}/collision/link1.STL" />
         </geometry>
       </collision>
@@ -219,5 +220,5 @@
         <geometry>
           <mesh
-            filename="package://robofox/meshes/awtube3_link2.STL" />
+            filename="package://ibt_ros2_description/meshes/${robofox_type}/visual/link2.STL" />
         </geometry>
         <material
@@ -233,5 +234,5 @@
         <geometry>
           <mesh
-            filename="package://robofox/meshes/controllo/awtube3_link2.STL" />
+            filename="package://ibt_ros2_description/meshes/${robofox_type}/collision/link2.STL" />
         </geometry>
       </collision>
@@ -279,5 +280,5 @@
         <geometry>
           <mesh
-            filename="package://robofox/meshes/awtube3_link3.STL" />
+            filename="package://ibt_ros2_description/meshes/${robofox_type}/visual/link3.STL" />
         </geometry>
         <material
@@ -293,5 +294,5 @@
         <geometry>
           <mesh
-            filename="package://robofox/meshes/controllo/awtube3_link3.STL" />
+            filename="package://ibt_ros2_description/meshes/${robofox_type}/collision/link3.STL" />
         </geometry>
       </collision>
@@ -339,5 +340,5 @@
         <geometry>
           <mesh
-            filename="package://robofox/meshes/awtube3_link4.STL" />
+            filename="package://ibt_ros2_description/meshes/${robofox_type}/visual/link4.STL" />
         </geometry>
         <material
@@ -353,5 +354,5 @@
         <geometry>
           <mesh
-            filename="package://robofox/meshes/controllo/awtube3_link4.STL" />
+            filename="package://ibt_ros2_description/meshes/${robofox_type}/collision/link4.STL" />
         </geometry>
       </collision>
@@ -399,5 +400,5 @@
         <geometry>
           <mesh
-            filename="package://robofox/meshes/awtube3_link5.STL" />
+            filename="package://ibt_ros2_description/meshes/${robofox_type}/visual/link5.STL" />
         </geometry>
         <material
@@ -413,5 +414,5 @@
         <geometry>
           <mesh
-            filename="package://robofox/meshes/controllo/awtube3_link5.STL" />
+            filename="package://ibt_ros2_description/meshes/${robofox_type}/collision/link5.STL" />
         </geometry>
       </collision>
@@ -459,5 +460,5 @@
         <geometry>
           <mesh
-            filename="package://robofox/meshes/awtube3_link6.STL" />
+            filename="package://ibt_ros2_description/meshes/${robofox_type}/visual/link6.STL" />
         </geometry>
         <material
@@ -473,5 +474,5 @@
         <geometry>
           <mesh
-            filename="package://robofox/meshes/controllo/awtube3_link6.STL" />
+            filename="package://ibt_ros2_description/meshes/${robofox_type}/collision/link6.STL" />
         </geometry>
       </collision>

Commit message: updated namespace

File: xacro/robofox.urdf (robot description, URDF)
Before this commit: robot robofox, 7 links, 6 joints
Links:
- link robofox_base_link: geometry 
- link robofox_link1: geometry 
- link robofox_link2: geometry 
- link robofox_link3: geometry 
- link robofox_link4: geometry 
- link robofox_link5: geometry 
- link robofox_link6: geometry 

File: xacro/robofox.urdf.xacro (robot description, xacro)
@@ -2,5 +2,5 @@
 <robot xmlns:xacro="http://wiki.ros.org/xacro" name="robofox">
     <xacro:arg name="prefix" default="robofox" />
-    <xacro:arg name="robofox_type" default="61814v3" />
+    <xacro:arg name="robofox_type" default="robofox_61814v3" />
     <xacro:arg name="physical_params_file"
         default="$(find ibt_ros2_description)/config/$(arg robofox_type)/physical_parameters.yaml" />
@@ -9,4 +9,5 @@
         prefix="$(arg prefix)"
         physical_params_file="$(arg physical_params_file)"
+        robofox_type="$(arg robofox_type)"
     >
         <origin xyz="0 0 0" rpy="0 0 0" />

File: xacro/robofox.xacro (robot description, xacro)
@@ -5,5 +5,5 @@
     params="
     prefix:='robofox'
-    robofox_type:='61814v3'
+    robofox_type:='robofox_61814v3'
     connected_to:=''
     *origin
@@ -134,6 +134,6 @@
           rpy="0 0 0" />
         <geometry>
-          <mesh
-            filename="package://ibt_ros2_description/meshes/${robofox_type}/collision/baselink.STL" />
+          <!-- <mesh
+            filename="package://ibt_ros2_description/meshes/${robofox_type}/collision/baselink.STL" /> -->
         </geometry>
       </collision>
@@ -156,5 +156,5 @@
       <visual>
         <origin
-          xyz="0 0 0.119"
+          xyz="0 0 -0.09"
           rpy="0 0 0" />
         <geometry>
@@ -173,6 +173,6 @@
           rpy="0 0 0" />
         <geometry>
-          <mesh
-            filename="package://ibt_ros2_description/meshes/${robofox_type}/collision/link1.STL" />
+          <!-- <mesh
+            filename="package://ibt_ros2_description/meshes/${robofox_type}/collision/link1.STL" /> -->
         </geometry>
       </collision>
@@ -217,22 +217,22 @@
         <origin
           xyz="0 0 0"
+          rpy="0 -${pi/2} 0" />
+        <geometry>
+          <!-- <mesh
+            filename="package://ibt_ros2_description/meshes/${robofox_type}/visual/link2.STL" /> -->
+        </geometry>
+        <material
+          name="">
+          <color
+            rgba="0.79216 0.81961 0.93333 1" />
+        </material>
+      </visual>
+      <collision>
+        <origin
+          xyz="0 0 0"
           rpy="-${pi/2.0} -${pi/2.0} 0" />
         <geometry>
-          <mesh
-            filename="package://ibt_ros2_description/meshes/${robofox_type}/visual/link2.STL" />
-        </geometry>
-        <material
-          name="">
-          <color
-            rgba="0.79216 0.81961 0.93333 1" />
-        </material>
-      </visual>
-      <collision>
-        <origin
-          xyz="0 0 0"
-          rpy="-${pi/2.0} -${pi/2.0} 0" />
-        <geometry>
-          <mesh
-            filename="package://ibt_ros2_description/meshes/${robofox_type}/collision/link2.STL" />
+          <!-- <mesh
+            filename="package://ibt_ros2_description/meshes/${robofox_type}/collision/link2.STL" /> -->
         </geometry>
       </collision>
@@ -279,6 +279,6 @@
           rpy="0 0 ${pi}" />
         <geometry>
-          <mesh
-            filename="package://ibt_ros2_description/meshes/${robofox_type}/visual/link3.STL" />
+          <!-- <mesh
+            filename="package://ibt_ros2_description/meshes/${robofox_type}/visual/link3.STL" /> -->
         </geometry>
         <material
@@ -293,6 +293,6 @@
           rpy="0 0 ${pi}" />
         <geometry>
-          <mesh
-            filename="package://ibt_ros2_description/meshes/${robofox_type}/collision/link3.STL" />
+          <!-- <mesh
+            filename="package://ibt_ros2_description/meshes/${robofox_type}/collision/link3.STL" /> -->
         </geometry>
       </collision>
@@ -339,6 +339,6 @@
           rpy="${pi/2.0} 0 0" />
         <geometry>
-          <mesh
-            filename="package://ibt_ros2_description/meshes/${robofox_type}/visual/link4.STL" />
+          <!-- <mesh
+            filename="package://ibt_ros2_description/meshes/${robofox_type}/visual/link4.STL" /> -->
         </geometry>
         <material
@@ -353,6 +353,6 @@
           rpy="${pi/2.0} 0 0" />
         <geometry>
-          <mesh
-            filename="package://ibt_ros2_description/meshes/${robofox_type}/collision/link4.STL" />
+          <!-- <mesh
+            filename="package://ibt_ros2_description/meshes/${robofox_type}/collision/link4.STL" /> -->
         </geometry>
       </collision>
@@ -399,6 +399,6 @@
           rpy="-${pi/2.0} ${pi/2.0} 0" />
         <geometry>
-          <mesh
-            filename="package://ibt_ros2_description/meshes/${robofox_type}/visual/link5.STL" />
+          <!-- <mesh
+            filename="package://ibt_ros2_description/meshes/${robofox_type}/visual/link5.STL" /> -->
         </geometry>
         <material
@@ -413,6 +413,6 @@
           rpy="-${pi/2.0} ${pi/2.0} 0" />
         <geometry>
-          <mesh
-            filename="package://ibt_ros2_description/meshes/${robofox_type}/collision/link5.STL" />
+          <!-- <mesh
+            filename="package://ibt_ros2_description/meshes/${robofox_type}/collision/link5.STL" /> -->
         </geometry>
       </collision>
@@ -459,6 +459,6 @@
           rpy="${pi/2.0} ${pi} 0" />
         <geometry>
-          <mesh
-            filename="package://ibt_ros2_description/meshes/${robofox_type}/visual/link6.STL" />
+          <!-- <mesh
+            filename="package://ibt_ros2_description/meshes/${robofox_type}/visual/link6.STL" /> -->
         </geometry>
         <material
@@ -473,6 +473,6 @@
           rpy="${pi/2.0} ${pi} 0" />
         <geometry>
-          <mesh
-            filename="package://ibt_ros2_description/meshes/${robofox_type}/collision/link6.STL" />
+          <!-- <mesh
+            filename="package://ibt_ros2_description/meshes/${robofox_type}/collision/link6.STL" /> -->
         </geometry>
       </collision>

Commit message: parameters fixed

File: xacro/robofox.urdf (robot description, URDF)
Before this commit: robot robofox, 7 links, 6 joints
Links:
- link robofox_base_link: geometry collision mesh filename=package://ibt_ros2_description/meshes/robofox_61814v3/visua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; visual mesh filename=package://ibt_ros2_description/meshes/robofox_61814v3/visua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
- link robofox_link1: geometry collision mesh filename=package://ibt_ros2_description/meshes/robofox_61814v3/visua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; visual mesh filename=package://ibt_ros2_description/meshes/robofox_61814v3/visua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
- link robofox_link2: geometry collision mesh filename=package://ibt_ros2_description/meshes/robofox_61814v3/visua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; visual mesh filename=package://ibt_ros2_description/meshes/robofox_61814v3/visua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
- link robofox_link3: geometry collision mesh filename=package://ibt_ros2_description/meshes/robofox_61814v3/visua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; visual mesh filename=package://ibt_ros2_description/meshes/robofox_61814v3/visua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
- link robofox_link4: geometry collision mesh filename=package://ibt_ros2_description/meshes/robofox_61814v3/visua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; visual mesh filename=package://ibt_ros2_description/meshes/robofox_61814v3/visua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
- link robofox_link5: geometry collision mesh filename=package://ibt_ros2_description/meshes/robofox_61814v3/visua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; visual mesh filename=package://ibt_ros2_description/meshes/robofox_61814v3/visua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
- link robofox_link6: geometry collision mesh filename=package://ibt_ros2_description/meshes/robofox_61814v3/visua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; visual mesh filename=package://ibt_ros2_description/meshes/robofox_61814v3/visua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
Joints:
- joint robofox_joint1: limit lower=-3.141592653589793 upper=3.141592653589793 effort=600 velocity=1.2436 -> lower=-3.14 upper=3.14 effort=600 velocity=1.2436
- joint robofox_joint2: limit lower=-3.141592653589793 upper=3.141592653589793 effort=690 velocity=0.86 -> lower=-3.14 upper=3.14 effort=690 velocity=0.86
- joint robofox_joint3: limit lower=-4.71 upper=4.71 effort=350 velocity=1.24 -> lower=-3.14 upper=3.14 effort=350 velocity=1.24
- joint robofox_joint4: limit lower=-8.0 upper=8.0 effort=145 velocity=2.71 -> lower=-3.14 upper=3.14 effort=145 velocity=2.71
- joint robofox_joint5: limit lower=-4.71 upper=4.71 effort=145 velocity=2.71 -> lower=-3.14 upper=3.14 effort=145 velocity=2.71
- joint robofox_joint6: limit lower=-8.0 upper=8.0 effort=85 velocity=3.61 -> lower=-3.14 upper=3.14 effort=85 velocity=3.61
