Commit message: AMR direction fixed

File: xacro/amr/amr.urdf.xacro (robot description, xacro)
@@ -2,5 +2,5 @@
 <robot xmlns:xacro="http://www.ros.org/wiki/xacro" name="amr">
     <xacro:include filename="$(find ibt_ros2_description)/xacro/amr/amr.xacro" />
-    <xacro:amr name="base_footprint" parent="base_link">
+    <xacro:amr>
         <origin xyz="0 0 0" rpy="0 0 0" />
     </xacro:amr>

File: xacro/amr/amr.xacro (robot description, xacro)
@@ -2,750 +2,753 @@
 <robot
   name="amr" xmlns:xacro="http://ros.org/wiki/xacro">
-  <xacro:macro name="amr" params="name parent *origin">
-    <joint name="${name}_joint" type="fixed">
-      <parent link="${parent}" />
-      <child link="${name}" />
-      <xacro:insert_block name="origin" />
-    </joint>
-    <link
-      name="base_link">
-      <inertial>
-        <origin
-          xyz="0.0019401 -0.00020197 0.43265"
-          rpy="0 0 0" />
-        <mass
-          value="95.371" />
-        <inertia
-          ixx="7.0414"
-          ixy="-0.0020566"
-          ixz="-0.14914"
-          iyy="7.048"
-          iyz="0.00016602"
-          izz="12.614" />
-      </inertial>
-      <visual>
-        <origin
-          xyz="0 0 0"
-          rpy="0 0 0" />
-        <geometry>
-          <mesh
-            filename="package://ibt_ros2_description/meshes/amr/base_link.STL" />
-        </geometry>
-        <material
-          name="">
-          <color
-            rgba="0.77647 0.75686 0.73725 1" />
-        </material>
-      </visual>
-      <collision>
-        <origin
-          xyz="0 0 0"
-          rpy="0 0 0" />
-        <geometry>
-          <mesh
-            filename="package://ibt_ros2_description/meshes/amr/base_link.STL" />
-        </geometry>
-      </collision>
-    </link>
-    <link
-      name="base_footprint">
-      <inertial>
-        <origin
-          xyz="0.00030419 0.00097233 0.2973"
-          rpy="0 0 0" />
-        <mass
-          value="27.996" />
-        <inertia
-          ixx="1.1622"
-          ixy="0.00018417"
-          ixz="9.0657E-07"
-          iyy="1.2308"
-          iyz="-1.2244E-06"
-          izz="2.3922" />
-      </inertial>
-      <visual>
-        <origin
-          xyz="0 0 0"
-          rpy="0 0 0" />
-        <geometry>
-          <mesh
-            filename="package://ibt_ros2_description/meshes/amr/base_footprint.STL" />
-        </geometry>
-        <material
-          name="">
-          <color
-            rgba="0.86667 0.86667 0.8902 1" />
-        </material>
-      </visual>
-      <collision>
-        <origin
-          xyz="0 0 0"
-          rpy="0 0 0" />
-        <geometry>
-          <mesh
-            filename="package://ibt_ros2_description/meshes/amr/base_footprint.STL" />
-        </geometry>
-      </collision>
-    </link>
-    <joint
-      name="base_footprint"
-      type="fixed">
-      <origin
-        xyz="0 0 0"
-        rpy="0 0 0" />
-      <parent
-        link="base_link" />
-      <child
-        link="base_footprint" />
-      <axis
-        xyz="0 0 0" />
-    </joint>
-    <link
-      name="mpo_700_caster_front_left_link">
-      <inertial>
-        <origin
-          xyz="5.5511E-17 0.0079242 -0.027057"
-          rpy="0 0 0" />
-        <mass
-          value="17.529" />
-        <inertia
-          ixx="0.15365"
-          ixy="-1.93E-18"
-          ixz="-2.0686E-17"
-          iyy="0.15493"
-          iyz="0.010987"
-          izz="0.025283" />
-      </inertial>
-      <visual>
-        <origin
-          xyz="0 0 0"
-          rpy="0 0 0" />
-        <geometry>
-          <mesh
-            filename="package://ibt_ros2_description/meshes/amr/mpo_700_caster_front_left_link.STL" />
-        </geometry>
-        <material
-          name="">
-          <color
-            rgba="0.77647 0.75686 0.73725 1" />
-        </material>
-      </visual>
-      <collision>
-        <origin
-          xyz="0 0 0"
-          rpy="0 0 0" />
-        <geometry>
-          <mesh
-            filename="package://ibt_ros2_description/meshes/amr/mpo_700_caster_front_left_link.STL" />
-        </geometry>
-      </collision>
-    </link>
-    <joint
-      name="mpo_700_caster_front_left_joint"
-      type="revolute">
-      <origin
-        xyz="0.26 0.26 0.22"
-        rpy="0 0 ${pi}" />
-      <parent
-        link="base_footprint" />
-      <child
-        link="mpo_700_caster_front_left_link" />
-      <axis
-        xyz="0 0 1" />
-      <limit
-        lower="-1E+16"
-        upper="1E+16"
-        effort="1000"
-        velocity="6.5" />
-      <dynamics
-        damping="30"
-        friction="110" />
-    </joint>
-    <link
-      name="mpo_700_wheel_front_left_link">
-      <inertial>
-        <origin
-          xyz="0 -0.015376 0"
-          rpy="0 0 0" />
-        <mass
-          value="5.9448" />
-        <inertia
-          ixx="0.012415"
-          ixy="-1.1866E-17"
-          ixz="-1.3603E-18"
-          iyy="0.02381"
-          iyz="-5.4807E-21"
-          izz="0.012415" />
-      </inertial>
-      <visual>
-        <origin
-          xyz="0 0 0"
-          rpy="0 0 0" />
-        <geometry>
-          <mesh
-            filename="package://ibt_ros2_description/meshes/amr/mpo_700_wheel_front_left_link.STL" />
-        </geometry>
-        <material
-          name="">
-          <color
-            rgba="0.77647 0.75686 0.73725 1" />
-        </material>
-      </visual>
-      <collision>
-        <origin
-          xyz="0 0 0"
-          rpy="0 0 0" />
-        <geometry>
-          <mesh
-            filename="package://ibt_ros2_description/meshes/amr/mpo_700_wheel_front_left_link.STL" />
-        </geometry>
-      </collision>
-    </link>
-    <joint
-      name="mpo_700_wheel_front_left_joint"
-      type="revolute">
-      <origin
-        xyz="0 -0.0603 -0.122"
-        rpy="0 0 3.1416" />
-      <parent
-        link="mpo_700_caster_front_left_link" />
-      <child
-        link="mpo_700_wheel_front_left_link" />
-      <axis
-        xyz="0 1 0" />
-      <limit
-        lower="-1E+16"
-        upper="1E+16"
-        effort="1000"
-        velocity="20.5" />
-      <dynamics
-        damping="30"
-        friction="110" />
-    </joint>
-    <link
-      name="mpo_700_caster_back_left_link">
-      <inertial>
-        <origin
-          xyz="-1.1102E-16 0.0079242 -0.027057"
-          rpy="0 0 0" />
-        <mass
-          value="17.529" />
-        <inertia
-          ixx="0.15365"
-          ixy="-1.6992E-18"
-          ixz="2.7876E-18"
-          iyy="0.15493"
-          iyz="0.010987"
-          izz="0.025283" />
-      </inertial>
-      <visual>
-        <origin
-          xyz="0 0 0"
-          rpy="0 0 0" />
-        <geometry>
-          <mesh
-            filename="package://ibt_ros2_description/meshes/amr/mpo_700_caster_back_left_link.STL" />
-        </geometry>
-        <material
-          name="">
-          <color
-            rgba="0.77647 0.75686 0.73725 1" />
-        </material>
-      </visual>
-      <collision>
-        <origin
-          xyz="0 0 0"
-          rpy="0 0 0" />
-        <geometry>
-          <mesh
-            filename="package://ibt_ros2_description/meshes/amr/mpo_700_caster_back_left_link.STL" />
-        </geometry>
-      </collision>
-    </link>
-    <joint
-      name="mpo_700_caster_back_left_joint"
-      type="revolute">
-      <origin
-        xyz="-0.26 0.26 0.22"
-        rpy="0 0 ${pi}" />
-      <parent
-        link="base_footprint" />
-      <child
-        link="mpo_700_caster_back_left_link" />
-      <axis
-        xyz="0 0 1" />
-      <limit
-        lower="-1E+16"
-        upper="1E+16"
-        effort="1000"
-        velocity="6.5" />
-      <dynamics
-        damping="30"
-        friction="110" />
-    </joint>
-    <link
-      name="mpo_700_wheel_back_left_link">
-      <inertial>
-        <origin
-          xyz="-5.5511E-17 -0.015376 0"
-          rpy="0 0 0" />
-        <mass
-          value="5.9448" />
-        <inertia
-          ixx="0.012415"
-          ixy="2.1868E-20"
-          ixz="-1.0384E-18"
-          iyy="0.02381"
-          iyz="-4.5314E-19"
-          izz="0.012415" />
-      </inertial>
-      <visual>
-        <origin
-          xyz="0 0 0"
-          rpy="0 0 0" />
-        <geometry>
-          <mesh
-            filename="package://ibt_ros2_description/meshes/amr/mpo_700_wheel_back_left_link.STL" />
-        </geometry>
-        <material
-          name="">
-          <color
-            rgba="0.77647 0.75686 0.73725 1" />
-        </material>
-      </visual>
-      <collision>
-        <origin
-          xyz="0 0 0"
-          rpy="0 0 0" />
-        <geometry>
-          <mesh
-            filename="package://ibt_ros2_description/meshes/amr/mpo_700_wheel_back_left_link.STL" />
-        </geometry>
-      </collision>
-    </link>
-    <joint
-      name="mpo_700_wheel_back_left_joint"
-      type="revolute">
-      <origin
-        xyz="0 -0.0603 -0.122"
-        rpy="0 0 -3.1416" />
-      <parent
-        link="mpo_700_caster_back_left_link" />
-      <child
-        link="mpo_700_wheel_back_left_link" />
-      <axis
-        xyz="0 1 0" />
-      <limit
-        lower="-1E+16"
-        upper="1E+16"
-        effort="1000"
-        velocity="20.5" />
-      <dynamics
-        damping="30"
-        friction="110" />
-    </joint>
-    <link
-      name="mpo_700_caster_front_right_link">
-      <inertial>
-        <origin
-          xyz="5.5511E-17 0.0079242 -0.027057"
-          rpy="0 0 0" />
-        <mass
-          value="17.529" />
-        <inertia
-          ixx="0.15365"
-          ixy="-1.8032E-18"
-          ixz="4.3901E-18"
-          iyy="0.15493"
-          iyz="0.010987"
-          izz="0.025283" />
-      </inertial>
-      <visual>
-        <origin
-          xyz="0 0 0"
-          rpy="0 0 0" />
-        <geometry>
-          <mesh
-            filename="package://ibt_ros2_description/meshes/amr/mpo_700_caster_front_right_link.STL" />
-        </geometry>
-        <material
-          name="">
-          <color
-            rgba="0.77647 0.75686 0.73725 1" />
-        </material>
-      </visual>
-      <collision>
-        <origin
-          xyz="0 0 0"
-          rpy="0 0 0" />
-        <geometry>
-          <mesh
-            filename="package://ibt_ros2_description/meshes/amr/mpo_700_caster_front_right_link.STL" />
-        </geometry>
-      </collision>
-    </link>
-    <joint
-      name="mpo_700_caster_front_right_joint"
-      type="revolute">
-      <origin
-        xyz="0.26 -0.26 0.22"
-        rpy="0 0 0" />
-      <parent
-        link="base_footprint" />
-      <child
-        link="mpo_700_caster_front_right_link" />
-      <axis
-        xyz="0 0 1" />
-      <limit
-        lower="-1E+16"
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
Commit message: camera for docking added

File: xacro/amr/amr.urdf.xacro (robot description, xacro)
@@ -5,3 +5,14 @@
         <origin xyz="0 0 0" rpy="0 0 0" />
     </xacro:amr>
+    <!-- Camera for docking -->
+    <xacro:arg name="use_nominal_extrinsics" default="false" />
+    <xacro:arg name="add_plug" default="false" />
+    <xacro:arg name="use_mesh" default="true" />
+    <xacro:include filename="$(find realsense2_description)/urdf/_d415.urdf.xacro" />
+    <xacro:sensor_d415 parent="camera_docking_mount"
+        use_nominal_extrinsics="$(arg use_nominal_extrinsics)"
+        add_plug="$(arg add_plug)"
+        use_mesh="$(arg use_mesh)">
+        <origin xyz="0 0 0" rpy="0 0 0" />
+    </xacro:sensor_d415>
 </robot>

File: xacro/amr/amr.xacro (robot description, xacro)
@@ -751,4 +751,21 @@
       xyz="0 0 0" />
   </joint>
+  <!-- Link for the docking camera -->
+  <link
+    name="${amr_prefix}camera_docking_mount">
+  </link>
+  <joint
+    name="${amr_prefix}camera_docking_mount"
+    type="fixed">
+    <origin
+        xyz="0 -0.4105 0.1195"
+        rpy="0 0 -1.57" />
+    <parent
+      link="${amr_prefix}base_link" />
+    <child
+      link="${amr_prefix}camera_docking_mount" />
+    <axis
+      xyz="0 0 0" />
+  </joint>
   </xacro:macro>
 </robot>

Commit message: link for the calibration camera

File: xacro/amr/amr.urdf.xacro (robot description, xacro)
@@ -16,3 +16,8 @@
         <origin xyz="0 0 0" rpy="0 0 0" />
     </xacro:sensor_d415>
+    <!-- Camera for calibration -->
+    <!-- <xacro:include filename="$(find realsense2_description)/urdf/_d435i.urdf.xacro"/>
+    <xacro:sensor_d435i parent="camera_calibration_mount" use_nominal_extrinsics="$(arg use_nominal_extrinsics)">
+        <origin xyz="0 0 0" rpy="0 0 0"/>
+    </xacro:sensor_d435i> -->
 </robot>

File: xacro/amr/amr.xacro (robot description, xacro)
@@ -768,4 +768,21 @@
       xyz="0 0 0" />
   </joint>
+  <!-- Link for the calibration camera -->
+  <link
+    name="${amr_prefix}camera_calibration_mount">
+  </link>
+  <joint
+    name="${amr_prefix}camera_calibration_mount"
+    type="fixed">
+    <origin
+        xyz="-0.45105 0.0 0.2825"
+        rpy="0 0 ${pi}" />
+    <parent
+      link="${amr_prefix}base_link" />
+    <child
+      link="${amr_prefix}camera_calibration_mount" />
+    <axis
+      xyz="0 0 0" />
+  </joint>
   </xacro:macro>
 </robot>

Commit message: added cameras

File: xacro/amr/amr.urdf.xacro (robot description, xacro)
@@ -6,5 +6,5 @@
     </xacro:amr>
     <!-- Camera for docking -->
-    <xacro:arg name="use_nominal_extrinsics" default="false" />
+    <!-- <xacro:arg name="use_nominal_extrinsics" default="false" />
     <xacro:arg name="add_plug" default="false" />
     <xacro:arg name="use_mesh" default="true" />
@@ -15,5 +15,5 @@
         use_mesh="$(arg use_mesh)">
         <origin xyz="0 0 0" rpy="0 0 0" />
-    </xacro:sensor_d415>
+    </xacro:sensor_d415> -->
     <!-- Camera for calibration -->
     <!-- <xacro:include filename="$(find realsense2_description)/urdf/_d435i.urdf.xacro"/>

File: xacro/amr/amr.xacro (robot description, xacro)
@@ -776,6 +776,6 @@
     type="fixed">
     <origin
-        xyz="-0.45105 0.0 0.2825"
-        rpy="0 0 ${pi}" />
+        xyz="0.45105 0.0 0.2825"
+        rpy="0 0 0" />
     <parent
       link="${amr_prefix}base_link" />

File: xacro/combofox/combofox.urdf.xacro (robot description, xacro)
@@ -1,5 +1,5 @@
 <?xml version="1.0" encoding="utf-8"?>
 <robot xmlns:xacro="http://www.ros.org/wiki/xacro" name="amr">
-    <!-- Arguments for robofox -->
+    <!-- Arguments -->
     <xacro:arg name="arm_prefix" default="robofox" />
     <xacro:arg name="arm_type" default="robofox_61814v3" />
@@ -8,8 +8,24 @@
     <xacro:arg name="joint_limits_file"
         default="$(find ibt_ros2_description)/config/$(arg arm_type)/joint_limits.yaml" />
+    <xacro:arg name="use_nominal_extrinsics" default="false" />
+    <xacro:arg name="camera_name" default="d435i" />
+	<!--xacro:arg name="parent_frame" default="GRIPPER" /-->
+    <!-- TODO: update position values -->
+	<xacro:arg name="cam_pos_x" default="0" />
+	<xacro:arg name="cam_pos_y" default="0.13204" />
+	<xacro:arg name="cam_pos_z" default="-0.0660" />
+	<xacro:arg name="cam_roll" default="3.1416" />
+	<xacro:arg name="cam_pitch" default="-1.5708" />
+	<xacro:arg name="cam_yaw" default="1.5708" />
+	<xacro:arg name="has_imu" default="false" />
     <!-- Amr combo base -->
     <xacro:include filename="$(find ibt_ros2_description)/xacro/amr/amr.xacro" />
     <!-- Robotic arm -->
     <xacro:include filename="$(find ibt_ros2_description)/xacro/robofox/robofox.xacro" />
+    <!-- Gripper -->
+    <xacro:include filename="$(find grip_exon)/urdf/grip_exon.urdf.xacro" />
+    <!-- Camera -->
+    <xacro:include filename="$(find realsense2_description)/urdf/_d435i.urdf.xacro"/>
+    <xacro:include filename="$(find realsense2_description)/urdf/_d435.urdf.xacro"/>
     <!-- Instances -->
     <xacro:amr>
@@ -25,3 +41,17 @@
         <origin xyz="0 0 0" rpy="0 0 ${pi/2}" />
     </xacro:robofox>
+  <xacro:grip_exon parent="robofox_link6">
+    <origin xyz="0 0 0" rpy="0 0 ${pi/2}"/>
+  </xacro:grip_exon>
+    <!-- Camera for arm -->
+    <xacro:sensor_d435
+        name="$(arg camera_name)"
+        parent="GRIPPER"
+    >
+        <origin xyz="$(arg cam_pos_x) $(arg cam_pos_y) $(arg cam_pos_z)" rpy="$(arg cam_roll) $(arg cam_pitch) $(arg cam_yaw)" />
+    </xacro:sensor_d435>
+    <!-- Camera for calibration of the base -->
+    <xacro:sensor_d435i parent="camera_calibration_mount" use_nominal_extrinsics="$(arg use_nominal_extrinsics)">
+        <origin xyz="0 0 0" rpy="0 0 0"/>
+    </xacro:sensor_d435i>
 </robot>
