Commit message: default value

File: xacro/amr/amr.xacro (robot description, xacro)
@@ -2,5 +2,5 @@
 <robot
   name="amr" xmlns:xacro="http://ros.org/wiki/xacro">
-  <xacro:macro name="amr" params="amr_prefix connected_to:='' *origin">
+  <xacro:macro name="amr" params="amr_prefix:='' connected_to:='' *origin">
     <!-- virtual joint -->
     <xacro:unless value="${not connected_to}">

File: xacro/combofox/combofox.urdf.xacro (robot description, xacro)
@@ -13,5 +13,5 @@
     <xacro:include filename="$(find ibt_ros2_description)/xacro/robofox/robofox.xacro" />
     <!-- Instances -->
-    <xacro:amr name="base_footprint" parent="base_link">
+    <xacro:amr>
         <origin xyz="0 0 0" rpy="0 0 0" />
     </xacro:amr>

Commit message: amr camera changed position

File: xacro/amr/amr.xacro (robot description, xacro)
@@ -759,6 +759,6 @@
     type="fixed">
     <origin
-        xyz="0 -0.4105 0.1195"
-        rpy="0 0 -1.57" />
+        xyz="0 0.4105 0.1195"
+        rpy="0 0 1.57" />
     <parent
       link="${amr_prefix}base_link" />

File: xacro/combofox/combofox.urdf.xacro (robot description, xacro)
@@ -12,8 +12,5 @@
     <!-- Robotic arm -->
     <xacro:include filename="$(find ibt_ros2_description)/xacro/robofox/robofox.xacro" />
-    <!-- Tray Gripper -->
-    <xacro:include filename="$(find tray_gripper)/xacro/tray_gripper.xacro" />
-    <!-- Camera Tray Gripper -->
-    <xacro:include filename="$(find camera_tray)/xacro/camera_tray.xacro" />
+    <!-- Gripper -->
     <!-- Realsense D415 camera -->
     <xacro:arg name="use_nominal_extrinsics" default="false" />
@@ -35,16 +32,4 @@
         <origin xyz="0 0 0" rpy="0 0 ${pi/2}" />
     </xacro:robofox>
-    <!-- Gripper -->
-    <xacro:tray_gripper
-        connected_to="robofox_link6"
-    >
-        <origin xyz="0 0 0" rpy="0 0 1.57" />
-    </xacro:tray_gripper>
-    <!-- Camera Gripper -->
-    <xacro:camera_tray
-        connected_to="tray_gripper_camera"
-    >
-        <origin xyz="0 0 0" rpy="0 0 0" />
-    </xacro:camera_tray>
     <!-- Camera docking -->
     <xacro:sensor_d415 parent="camera_docking_mount"
