Commit message: combofox display fixed

File: xacro/combofox/combofox.urdf.xacro (robot description, xacro)
@@ -1,4 +1,5 @@
-<?xml version="1.0"?>
-<robot xmlns:xacro="http://wiki.ros.org/xacro" name="robofox">
+<?xml version="1.0" encoding="utf-8"?>
+<robot xmlns:xacro="http://www.ros.org/wiki/xacro" name="amr">
+    <!-- Arguments for robofox -->
     <xacro:arg name="arm_prefix" default="robofox" />
     <xacro:arg name="arm_type" default="robofox_61814v3" />
@@ -7,12 +8,20 @@
     <xacro:arg name="joint_limits_file"
         default="$(find ibt_ros2_description)/config/$(arg arm_type)/joint_limits.yaml" />
+    <!-- Amr combo base -->
+    <xacro:include filename="$(find ibt_ros2_description)/xacro/amr/amr.xacro" />
+    <!-- Robotic arm -->
     <xacro:include filename="$(find ibt_ros2_description)/xacro/robofox/robofox.xacro" />
+    <!-- Instances -->
+    <xacro:amr name="base_footprint" parent="base_link">
+        <origin xyz="0 0 0" rpy="0 0 0" />
+    </xacro:amr>
     <xacro:robofox
-        arm_prefix="$(arg arm_prefix)"
+        arm_prefix="robofox"
         physical_params_file="$(arg physical_params_file)"
         joint_limits_file="$(arg joint_limits_file)"
         arm_type="$(arg arm_type)"
+        connected_to="agv_link1"
     >
-        <origin xyz="0 0 0" rpy="0 0 0" />
+        <origin xyz="0 0 0" rpy="0 0 ${pi/2}" />
     </xacro:robofox>
 </robot>

File: xacro/robofox/robofox.xacro (robot description, xacro)
@@ -4,6 +4,6 @@
   <xacro:macro name="robofox"
     params="
-    prefix:='robofox'
-    robofox_type:='robofox_61814v3'
+    arm_prefix:='robofox'
+    arm_type:='robofox_61814v3'
     connected_to:=''
     *origin
@@ -102,5 +102,5 @@
       <joint name="world" type="fixed">
         <parent link="${connected_to}" />
-        <child link="${prefix}_base_link" />
+        <child link="${arm_prefix}_base_link" />
         <xacro:insert_block name="origin" />
       </joint>
@@ -108,5 +108,5 @@
     <!-- chain -->
     <link
-      name="${prefix}_base_link">
+      name="${arm_prefix}_base_link">
       <inertial>
         <origin
@@ -128,24 +128,24 @@
         <geometry>
           <mesh
-            filename="package://ibt_ros2_description/meshes/${robofox_type}/visual/base_link.STL" />
-        </geometry>
-        <material
-          name="">
-          <color
-            rgba="0.30 0.30 0.30 1" />
-        </material>
-      </visual>
-      <collision>
-        <origin
-          xyz="0 0 0"
-          rpy="0 0 0" />
-        <geometry>
-          <mesh
-            filename="package://ibt_ros2_description/meshes/${robofox_type}/visual/base_link.STL" />
-        </geometry>
-      </collision>
-    </link>
-    <link
-      name="${prefix}_link1">
+            filename="package://ibt_ros2_description/meshes/${arm_type}/visual/base_link.STL" />
+        </geometry>
+        <material
+          name="">
+          <color
+            rgba="0.30 0.30 0.30 1" />
+        </material>
+      </visual>
+      <collision>
+        <origin
+          xyz="0 0 0"
+          rpy="0 0 0" />
+        <geometry>
+          <mesh
+            filename="package://ibt_ros2_description/meshes/${arm_type}/visual/base_link.STL" />
+        </geometry>
+      </collision>
+    </link>
+    <link
+      name="${arm_prefix}_link1">
       <inertial>
         <origin
@@ -167,24 +167,24 @@
         <geometry>
           <mesh
-            filename="package://ibt_ros2_description/meshes/${robofox_type}/visual/link1.STL" />
-        </geometry>
-        <material
-          name="">
-          <color
-            rgba="0.30 0.30 0.30 1" />
-        </material>
-      </visual>
-      <collision>
-        <origin
-          xyz="0 0 0"
-          rpy="0 0 0" />
-        <geometry>
-          <mesh
-            filename="package://ibt_ros2_description/meshes/${robofox_type}/visual/link1.STL" />
+            filename="package://ibt_ros2_description/meshes/${arm_type}/visual/link1.STL" />
+        </geometry>
+        <material
+          name="">
+          <color
+            rgba="0.30 0.30 0.30 1" />
+        </material>
+      </visual>
+      <collision>
+        <origin
+          xyz="0 0 0"
+          rpy="0 0 0" />
+        <geometry>
+          <mesh
+            filename="package://ibt_ros2_description/meshes/${arm_type}/visual/link1.STL" />
         </geometry>
       </collision>
     </link>
     <joint
-      name="${prefix}_joint1"
+      name="${arm_prefix}_joint1"
       type="revolute">
       <origin
@@ -192,7 +192,7 @@
         rpy="0 0 0" />
       <parent
-        link="${prefix}_base_link" />
+        link="${arm_prefix}_base_link" />
       <child
-        link="${prefix}_link1" />
+        link="${arm_prefix}_link1" />
       <axis
         xyz="0 0 -1" />
@@ -207,5 +207,5 @@
     </joint>
     <link
-      name="${prefix}_link2">
+      name="${arm_prefix}_link2">
       <inertial>
         <origin
@@ -227,24 +227,24 @@
         <geometry>
           <mesh
-            filename="package://ibt_ros2_description/meshes/${robofox_type}/visual/link2.STL" />
-        </geometry>
-        <material
-          name="">
-          <color
-            rgba="0.30 0.30 0.30 1" />
-        </material>
-      </visual>
-      <collision>
-        <origin
-          xyz="0 0 0"
-          rpy="0 0 0" />
-        <geometry>
-          <mesh
-            filename="package://ibt_ros2_description/meshes/${robofox_type}/visual/link2.STL" />
+            filename="package://ibt_ros2_description/meshes/${arm_type}/visual/link2.STL" />
+        </geometry>
+        <material
+          name="">
+          <color
+            rgba="0.30 0.30 0.30 1" />
+        </material>
+      </visual>
+      <collision>
+        <origin
+          xyz="0 0 0"
+          rpy="0 0 0" />
+        <geometry>
+          <mesh
+            filename="package://ibt_ros2_description/meshes/${arm_type}/visual/link2.STL" />
         </geometry>
       </collision>
     </link>
     <joint
-      name="${prefix}_joint2"
+      name="${arm_prefix}_joint2"
       type="revolute">
       <origin
@@ -252,7 +252,7 @@
         rpy="-${pi/2.0} -${pi/2.0} 0" />
       <parent
-        link="${prefix}_link1" />
+        link="${arm_prefix}_link1" />
       <child
-        link="${prefix}_link2" />
+        link="${arm_prefix}_link2" />
       <axis
         xyz="0 0 -1" />
@@ -267,5 +267,5 @@
     </joint>
     <link
-      name="${prefix}_link3">
+      name="${arm_prefix}_link3">
       <inertial>
         <origin
@@ -287,24 +287,24 @@
         <geometry>
           <mesh
-            filename="package://ibt_ros2_description/meshes/${robofox_type}/visual/link3.STL" />
-        </geometry>
-        <material
-          name="">
-          <color
-            rgba="0.30 0.30 0.30 1" />
-        </material>
-      </visual>
-      <collision>
-        <origin
-          xyz="0 0 0"
-          rpy="0 0 0" />
-        <geometry>
-          <mesh
-            filename="package://ibt_ros2_description/meshes/${robofox_type}/visual/link3.STL" />
+            filename="package://ibt_ros2_description/meshes/${arm_type}/visual/link3.STL" />
+        </geometry>
+        <material
+          name="">
+          <color
+            rgba="0.30 0.30 0.30 1" />
+        </material>
+      </visual>
+      <collision>
+        <origin
+          xyz="0 0 0"
+          rpy="0 0 0" />
+        <geometry>
+          <mesh
+            filename="package://ibt_ros2_description/meshes/${arm_type}/visual/link3.STL" />
         </geometry>
       </collision>
     </link>
     <joint
-      name="${prefix}_joint3"
+      name="${arm_prefix}_joint3"
       type="revolute">
       <origin
@@ -312,7 +312,7 @@
         rpy="0 0 ${pi}" />
       <parent
-        link="${prefix}_link2" />
+        link="${arm_prefix}_link2" />
       <child
-        link="${prefix}_link3" />
+        link="${arm_prefix}_link3" />
       <axis
         xyz="0 0 -1" />
@@ -327,5 +327,5 @@
     </joint>
     <link
-      name="${prefix}_link4">
+      name="${arm_prefix}_link4">
       <inertial>
         <origin
@@ -347,24 +347,24 @@
         <geometry>
           <mesh
-            filename="package://ibt_ros2_description/meshes/${robofox_type}/visual/link4.STL" />
-        </geometry>
-        <material
-          name="">
-          <color
-            rgba="0.30 0.30 0.30 1" />
-        </material>
-      </visual>
-      <collision>
-        <origin
-          xyz="0 0 0"
-          rpy="0 0 0" />
-        <geometry>
-          <mesh
-            filename="package://ibt_ros2_description/meshes/${robofox_type}/visual/link4.STL" />
+            filename="package://ibt_ros2_description/meshes/${arm_type}/visual/link4.STL" />
+        </geometry>
+        <material
+          name="">
+          <color
+            rgba="0.30 0.30 0.30 1" />
+        </material>
+      </visual>
+      <collision>
+        <origin
+          xyz="0 0 0"
+          rpy="0 0 0" />
+        <geometry>
+          <mesh
+            filename="package://ibt_ros2_description/meshes/${arm_type}/visual/link4.STL" />
         </geometry>
       </collision>
     </link>
     <joint
-      name="${prefix}_joint4"
+      name="${arm_prefix}_joint4"
       type="revolute">
       <origin
@@ -372,7 +372,7 @@
         rpy="${pi/2.0} 0 0" />
       <parent
-        link="${prefix}_link3" />
+        link="${arm_prefix}_link3" />
       <child
-        link="${prefix}_link4" />
+        link="${arm_prefix}_link4" />
       <axis
         xyz="0 0 -1" />
@@ -387,5 +387,5 @@
     </joint>
     <link
-      name="${prefix}_link5">
+      name="${arm_prefix}_link5">
       <inertial>
         <origin
@@ -407,24 +407,24 @@
         <geometry>
           <mesh
-            filename="package://ibt_ros2_description/meshes/${robofox_type}/visual/link5.STL" />
-        </geometry>
-        <material
-          name="">
-          <color
-            rgba="0.30 0.30 0.30 1" />
-        </material>
-      </visual>
-      <collision>
-        <origin
-          xyz="0 0 0"
-          rpy="0 0 0" />
-        <geometry>
-          <mesh
-            filename="package://ibt_ros2_description/meshes/${robofox_type}/visual/link5.STL" />
+            filename="package://ibt_ros2_description/meshes/${arm_type}/visual/link5.STL" />
+        </geometry>
+        <material
+          name="">
+          <color
+            rgba="0.30 0.30 0.30 1" />
+        </material>
+      </visual>
+      <collision>
+        <origin
+          xyz="0 0 0"
+          rpy="0 0 0" />
+        <geometry>
+          <mesh
+            filename="package://ibt_ros2_description/meshes/${arm_type}/visual/link5.STL" />
         </geometry>
       </collision>
     </link>
     <joint
-      name="${prefix}_joint5"
+      name="${arm_prefix}_joint5"
       type="revolute">
       <origin
@@ -432,7 +432,7 @@
         rpy="-${pi/2.0} ${pi/2.0} 0" />
       <parent
-        link="${prefix}_link4" />
+        link="${arm_prefix}_link4" />
       <child
-        link="${prefix}_link5" />
+        link="${arm_prefix}_link5" />
       <axis
         xyz="0 0 -1" />
@@ -447,5 +447,5 @@
     </joint>
     <link
-      name="${prefix}_link6">
+      name="${arm_prefix}_link6">
       <inertial>
         <origin
@@ -467,24 +467,24 @@
         <geometry>
           <mesh
-            filename="package://ibt_ros2_description/meshes/${robofox_type}/visual/link6.STL" />
-        </geometry>
-        <material
-          name="">
-          <color
-            rgba="0.30 0.30 0.30 1" />
-        </material>
-      </visual>
-      <collision>
-        <origin
-          xyz="0 0 0"
-          rpy="0 0 0" />
-        <geometry>
-          <mesh
-            filename="package://ibt_ros2_description/meshes/${robofox_type}/visual/link6.STL" />
+            filename="package://ibt_ros2_description/meshes/${arm_type}/visual/link6.STL" />
+        </geometry>
+        <material
+          name="">
+          <color
+            rgba="0.30 0.30 0.30 1" />
+        </material>
+      </visual>
+      <collision>
+        <origin
+          xyz="0 0 0"
+          rpy="0 0 0" />
+        <geometry>
+          <mesh
+            filename="package://ibt_ros2_description/meshes/${arm_type}/visual/link6.STL" />
         </geometry>
       </collision>
     </link>
     <joint
-      name="${prefix}_joint6"
+      name="${arm_prefix}_joint6"
       type="revolute">
       <origin
@@ -492,7 +492,7 @@
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
Commit message: update rotation of grip

File: xacro/combofox/combofox.urdf.xacro (robot description, xacro)
@@ -12,8 +12,18 @@
     <!-- Robotic arm -->
     <xacro:include filename="$(find ibt_ros2_description)/xacro/robofox/robofox.xacro" />
-    <!-- Instances -->
+    <!-- Tray Gripper -->
+    <xacro:include filename="$(find tray_gripper)/xacro/tray_gripper.xacro" />
+    <!-- Camera Tray Gripper -->
+    <xacro:include filename="$(find camera_tray)/xacro/camera_tray.xacro" />
+    <!-- Realsense D415 camera -->
+    <xacro:arg name="use_nominal_extrinsics" default="false" />
+    <xacro:arg name="add_plug" default="false" />
+    <xacro:arg name="use_mesh" default="false" />
+    <xacro:include filename="$(find realsense2_description)/urdf/_d415.urdf.xacro" />
+    <!-- ARM -->
     <xacro:amr>
         <origin xyz="0 0 0" rpy="0 0 0" />
     </xacro:amr>
+    <!-- Robofox -->
     <xacro:robofox
         arm_prefix="robofox"
@@ -25,3 +35,22 @@
         <origin xyz="0 0 0" rpy="0 0 ${pi/2}" />
     </xacro:robofox>
+    <!-- Gripper -->
+    <xacro:tray_gripper
+        connected_to="robofox_link6"
+    >
+        <origin xyz="0 0 0" rpy="0 0 1.57" />
+    </xacro:tray_gripper>
+    <!-- Camera Gripper -->
+    <xacro:camera_tray
+        connected_to="tray_gripper_camera"
+    >
+        <origin xyz="0 0 0" rpy="0 0 0" />
+    </xacro:camera_tray>
+    <!-- Camera docking -->
+    <xacro:sensor_d415 parent="camera_docking_mount"
+        use_nominal_extrinsics="$(arg use_nominal_extrinsics)"
+        add_plug="$(arg add_plug)"
+        use_mesh="$(arg use_mesh)">
+        <origin xyz="0 0 0" rpy="0 0 0" />
+    </xacro:sensor_d415>
 </robot>

Commit message: bucket gripper included

File: xacro/combofox/combofox.urdf.xacro (robot description, xacro)
@@ -12,5 +12,6 @@
     <!-- Robotic arm -->
     <xacro:include filename="$(find ibt_ros2_description)/xacro/robofox/robofox.xacro" />
-    <!-- Gripper -->
+    <!-- Bucket Gripper -->
+    <xacro:include filename="$(find bucket_gripper)/xacro/bucket_gripper.xacro" />
     <!-- Realsense D415 camera -->
     <xacro:arg name="use_nominal_extrinsics" default="false" />
@@ -32,4 +33,10 @@
         <origin xyz="0 0 0" rpy="0 0 ${pi/2}" />
     </xacro:robofox>
+    <!-- Gripper -->
+    <xacro:bucket_gripper
+        connected_to="robofox_link6"
+    >
+        <origin xyz="0 0 0" rpy="0 0 0" />
+    </xacro:bucket_gripper>
     <!-- Camera docking -->
     <xacro:sensor_d415 parent="camera_docking_mount"
